Commit message: [1.4.0] Added skid steering Gazebo plugin macro
Added a macro simplifying the use of the differential drive plugin for skid
steering mobile bases.

Signed-off-by: Helio Perroni Filho <xperroni@gmail.com>

File: urdf/gazebo.xacro (robot description, xacro)
@@ -129,4 +129,29 @@
     </gazebo>
   </xacro:macro>
+  <xacro:macro
+    name="skid_controller"
+    params="
+      name
+      publish_odom:=true
+      **joints
+      **wheels
+    "
+  >
+    <gazebo>
+      <plugin name="${name}_joint_states" filename="libgazebo_ros_joint_state_publisher.so">
+        <xacro:insert_block name="joints"/>
+      </plugin>
+      <plugin name="${name}_controller" filename="libgazebo_ros_diff_drive.so">
+        <xacro:insert_block name="wheels"/>
+        <update_rate>50</update_rate>
+        <max_wheel_torque>20</max_wheel_torque>
+        <max_wheel_acceleration>1.0</max_wheel_acceleration>
+        <odometry_frame>odom</odometry_frame>
+        <robot_base_frame>base_link</robot_base_frame>
+        <publish_odom>${publish_odom}</publish_odom>
+        <publish_odom_tf>${publish_odom}</publish_odom_tf>
+      </plugin>
+    </gazebo>
+  </xacro:macro>
   <!-- See: http://sdformat.org/tutorials?tut=sdformat_urdf_extensions&cat=specification -->
   <xacro:macro
